Commit message: wip figuring out lfs stuff

File: isaac_neuromeka/assets/model/urdf/indy7_simplified.urdf (robot description, URDF)
Before this commit: robot indy7, 8 links, 7 joints
Links:
- link link2: geometry collision capsule length=0.35 radius=0.075; visual mesh filename=package://indy7_visualization/meshes/stl/Indy7_2.stl
- link link3: geometry collision capsule length=0.18 radius=0.05; collision cylinder length=0.05 radius=0.05
- link link4: geometry collision cylinder length=0.15 radius=0.05; visual mesh filename=package://indy7_visualization/meshes/stl/Indy7_4.stl
- link link5: geometry collision cylinder length=0.2 radius=0.05; visual mesh filename=package://indy7_visualization/meshes/stl/Indy7_5.stl
